File: PCB/Handheld Gaming device PCB/Handheld Gaming device PCB.kicad_pcb (KiCad board)
At the start: 2 copper layers, 337.8 x 81.8 mm, 72 parts, among them J1 Conn_02x20_Odd_Even, J10 Connector Left Board, J11 Connector Right Board, J12 Connector Right Board, J13 Connector Left Board, J2 USB_C_Receptacle_USB2.0_14P, J3 Joystick_Left, J4 Joystick_Right, J5 Display_5V, J6 Speaker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

Commit message: changed the PCB to use the module instead of the chip
Parts:
- removed C1: 10µF, Capacitor_SMD:C_0805_2012Metric
- removed C2: 4.7µF, Capacitor_SMD:C_0805_2012Metric
- removed D1: RED, LED_THT:LED_D3.0mm
- removed D2: Green, LED_THT:LED_D3.0mm
- removed R1: 2K, Resistor_SMD:R_0402_1005Metric
- removed R16, R17: 5.1k, Resistor_SMD:R_0402_1005Metric
- removed R2, R3: 1K, Resistor_SMD:R_0402_1005Metric
- removed U1: TP4056-42-ESOP8, Package_SO:SOIC-8-1EP_3.9x4.9mm_P1.27mm_EP2.41x3.3mm_ThermalVias
- J10, J13: value Connector Left Board -> FCC Connector Left Board
- J11, J12: value Connector Right Board -> FCC Connector Right Board
- J2: value USB_C_Receptacle_USB2.0_14P -> TP4056_Module; footprint Connector_USB:USB_C_Receptacle_GCT_USB4085 -> Connector_PinHeader_2.54mm:PinHeader_1x02_P2.54mm_Vertical
- moved J2 17.8 mm to (480.0, 200.5), turned to 0 degrees
Routing:
- net /USB_5V: track 51.4 -> 0.00 mm
- net /VBAT+: track 95.7 -> 128.2 mm
- net Net-(D2-K): track 30.5 -> 0.00 mm, vias 2 -> 0
- net Net-(D1-K): track 28.6 -> 0.00 mm, vias 2 -> 0
- net Net-(U1-~{STDBY}): track 14.6 -> 0.00 mm
- net Net-(U1-~{CHRG}): track 12.6 -> 0.00 mm, vias 2 -> 0
- net Net-(U1-GND): track 9.05 -> 0.00 mm
- net Net-(U1-PROG): track 5.52 -> 0.00 mm
- net /JOY_R_X: track 225.8 -> 225.2 mm

Commit message: added art on my PCB including a capybara and a horse that i drew myself!!!
Parts:
- added G***: LOGO, LOGO, F.Cu at (481.5, 234.6)
