File: src/PCB/Panelised PCB/Handheld_Panel.kicad_sch (KiCad schematic)
At the start: 26 parts, among them J1 Conn_02x20_Odd_Even, J12 FCC Connector Right Board, J13 FCC Connector Left Board, J2 TP4056_Module, J5 Display_5V, J6 Speaker, J7 AudioJack3_3.5mm, SW1 SW_SPDT, U2 MT3608, U3 ADS1115IDGS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

Commit message: fixed errors in like the PCB that i just now noticed
Parts:
- C6: footprint Capacitor_SMD:C_0402_1005Metric -> Capacitor_SMD:C_0805_2012Metric
- R18, R19, R20, R21, R4, R5: footprint Resistor_SMD:R_0402_1005Metric -> Resistor_SMD:R_0805_2012Metric
