File: src/PCB/Panelised PCB/Handheld_Panel.kicad_pcb (KiCad board)
At the start: 2 copper layers, 337.8 x 95.8 mm, 60 parts, among them J1 Conn_02x20_Odd_Even, J12 FCC Connector Right Board, J13 FCC Connector Left Board, J2 TP4056_Module, J5 Display_5V, J6 Speaker, J7 AudioJack3_3.5mm, SW1 SW_SPDT, U2 MT3608, U3 ADS1115IDGS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

Commit message: fixed errors in like the PCB that i just now noticed
Parts:
- added J10: FCC Connector Left Board, Connector_PinHeader_1.00mm:PinHeader_1x12_P1.00mm_Vertical, F.Cu at (315.9, 61.5)
- added J11: FCC Connector Right Board, Connector_PinHeader_1.00mm:PinHeader_1x12_P1.00mm_Vertical, F.Cu at (526.1, 66.6)
- added J3: Joystick_Left, Connector_PinSocket_2.54mm:PinSocket_1x05_P2.54mm_Horizontal, F.Cu at (307.0, 38.6)
- added J4: Joystick_Right, Connector_PinSocket_2.54mm:PinSocket_1x05_P2.54mm_Horizontal, F.Cu at (537.7, 55.2)
- added R10: 10k, Resistor_SMD:R_0805_2012Metric, B.Cu at (293.8, 66.9)
- added R11: 10k, Resistor_SMD:R_0805_2012Metric, B.Cu at (280.2, 85.4)
- added R12: 10k, Resistor_SMD:R_0805_2012Metric, B.Cu at (269.9, 76.4)
- added R13: 10k, Resistor_SMD:R_0805_2012Metric, B.Cu at (303.1, 76.2)
- added R14: 10k, Resistor_SMD:R_0805_2012Metric, B.Cu at (311.2, 43.7)
- added R15: 10k, Resistor_SMD:R_0805_2012Metric, B.Cu at (311.1, 47.4)
- added R22: 10k, Resistor_SMD:R_0805_2012Metric, B.Cu at (267.9, 99.1)
- added R23: 10k, Resistor_SMD:R_0805_2012Metric, B.Cu at (305.1, 99.2)
- added R24: 20k, Resistor_SMD:R_0805_2012Metric, B.Cu at (315.7, 43.9)
- added R25: 20k, Resistor_SMD:R_0805_2012Metric, B.Cu at (315.7, 47.5)
- added R26: 20k, Resistor_SMD:R_0805_2012Metric, B.Cu at (527.1, 50.4)
- added R27: 20k, Resistor_SMD:R_0805_2012Metric, B.Cu at (527.0, 46.3)
- added R28: 10k, Resistor_SMD:R_0805_2012Metric, B.Cu at (532.5, 50.2)
- added R29: 10k, Resistor_SMD:R_0805_2012Metric, B.Cu at (532.0, 46.2)
- added R6: 10k, Resistor_SMD:R_0805_2012Metric, B.Cu at (549.9, 88.2)
- added R7: 10k, Resistor_SMD:R_0805_2012Metric, B.Cu at (573.0, 78.3)
- added R8: 10k, Resistor_SMD:R_0805_2012Metric, B.Cu at (540.4, 79.5)
- added R9: 10k, Resistor_SMD:R_0805_2012Metric, B.Cu at (549.5, 70.4)
- added SW12: Start, Button_Switch_THT:SW_PUSH_6mm_H5mm, F.Cu at (272.0, 96.5)
- added SW13: Select, Button_Switch_THT:SW_PUSH_6mm_H5mm, F.Cu at (295.3, 96.8)
- added SW2: Button_A, Button_Switch_THT:SW_PUSH_6mm_H5mm, F.Cu at (553.6, 85.2)
- added SW3: Button_B, Button_Switch_THT:SW_PUSH_6mm_H5mm, F.Cu at (562.9, 76.4)
- added SW4: Button_X, Button_Switch_THT:SW_PUSH_6mm_H5mm, F.Cu at (543.9, 76.7)
- added SW5: Button_Y, Button_Switch_THT:SW_PUSH_6mm_H5mm, F.Cu at (553.4, 67.9)
- added SW6: D-pad UP, Button_Switch_THT:SW_PUSH_6mm_H5mm, F.Cu at (283.5, 65.0)
- added SW7: D-pad DOWN, Button_Switch_THT:SW_PUSH_6mm_H5mm, F.Cu at (283.5, 83.0)
- added SW8: D-pad LEFT, Button_Switch_THT:SW_PUSH_6mm_H5mm, F.Cu at (273.5, 73.8)
- added SW9: D-pad RIGHT, Button_Switch_THT:SW_PUSH_6mm_H5mm, F.Cu at (293.2, 73.8)
- C6: footprint Capacitor_SMD:C_0402_1005Metric -> Capacitor_SMD:C_0805_2012Metric
- R18, R19, R20, R21, R4, R5: footprint Resistor_SMD:R_0402_1005Metric -> Resistor_SMD:R_0805_2012Metric
Routing:
- net (no net): track 1192.2 -> 0.00 mm, vias 21 -> 0
- net +3.3V: track 342.7 -> 691.0 mm
- net /Left_Daughter_Board/GPIO13: track 0.00 -> 101.8 mm, vias 0 -> 2
- net /Left_Daughter_Board/GPIO4: track 0.00 -> 82.2 mm
- net /Left_Daughter_Board/GPIO26: track 0.00 -> 73.9 mm
- net /Right_Daughter_Board/GPIO27: track 0.00 -> 69.2 mm, vias 0 -> 2
- net /Left_Daughter_Board/GPIO25: track 0.00 -> 54.7 mm, vias 0 -> 4
- net +5V: track 0.00 -> 53.7 mm
- net /Left_Daughter_Board/GPIO6: track 0.00 -> 51.3 mm, vias 0 -> 2
- net /Right_Daughter_Board/GPIO17: track 0.00 -> 49.4 mm, vias 0 -> 2
- net /Right_Daughter_Board/GPIO16: track 0.00 -> 43.3 mm
- net /Right_Daughter_Board/GPIO23: track 0.00 -> 42.3 mm, vias 0 -> 2
- net /Right_Daughter_Board/JOY_R_Y: track 0.00 -> 34.7 mm
- net /Left_Daughter_Board/GPIO5: track 0.00 -> 33.8 mm, vias 0 -> 2
- net /Left_Daughter_Board/JOY_L_X: track 0.00 -> 31.1 mm, vias 0 -> 1
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
Commit message: fixed stuff in the panelised PCB---> fixed the traces as many MANY were at like 90 degree angles and were kindoff messed up then also updated resistors and capacitors to 0805 size as i am planning on hand solder
Parts:
- removed the G*** at (310.4, 89.4)
- removed the G*** at (490.7, 60.6)
- added G***: LOGO, LOGO, F.Cu at (310.8, 91.8)
- added G***: LOGO, LOGO, F.Cu at (495.4, 42.7)
Routing:
- net /Left_Daughter_Board/GPIO26: track 73.9 -> 27.1 mm, vias 0 -> 1
- net /+5V: track 487.2 -> 457.6 mm
- net /VBAT+: track 128.2 -> 117.5 mm
- net /GPIO25: track 87.7 -> 79.0 mm
- net /Left_Daughter_Board/GPIO13: track 101.8 -> 93.3 mm
- net /I2C_SCL: track 34.7 -> 27.2 mm
- net +3.3V: track 691.0 -> 683.8 mm
- net /I2S_LRCLK: track 172.6 -> 165.7 mm
- net /JOY_R_Y: track 227.9 -> 222.2 mm, vias 8 -> 10
- net /Left_Daughter_Board/GPIO6: track 51.3 -> 45.8 mm
- net /JOY_R_X: track 225.2 -> 220.0 mm
- net /Left_Daughter_Board/GPIO25: track 54.7 -> 49.7 mm, vias 4 -> 3
- net /JOY_L_Y: track 25.2 -> 20.3 mm
- net /GPIO4: track 48.9 -> 44.9 mm
- net Net-(C8-Pad2): track 42.6 -> 39.5 mm
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